Commit message: Updated description files

File: description/ackermann.urdf.xacro (robot description, xacro)
@@ -3,6 +3,5 @@
     <!-- Main URDF file for Ackermann Drive Robot -->
     <!-- Include general xacro files -->
-    <xacro:include filename="inertials.xacro"/>
-    <xacro:include filename="materials.xacro"/>
+    <xacro:include filename="common.xacro"/>
     <!-- Include sensors -->
     <xacro:include filename="lidar.xacro"/>
@@ -62,5 +61,5 @@
         <origin xyz="${front_wheel_offset_x} ${wheel_offset_y} ${wheel_offset_z}" rpy="0 0 0" />
         <axis xyz="0 0 1" />
-        <limit upper="0.6" lower="-0.6" effort="-1.0" velocity="-1.0" />
+        <limit upper="0.8" lower="-0.8" effort="-1.0" velocity="-1.0" />
     </joint>
     <link name="front_left_steer">
@@ -81,5 +80,5 @@
         <origin xyz="${front_wheel_offset_x} ${-wheel_offset_y} ${wheel_offset_z}" rpy="0 0 0" />
         <axis xyz="0 0 1" />
-        <limit upper="0.6" lower="-0.6" effort="-1.0" velocity="-1.0" />
+        <limit upper="0.8" lower="-0.8" effort="-1.0" velocity="-1.0" />
     </joint>
     <link name="front_right_steer">
@@ -281,6 +280,6 @@
             <!-- Limits -->
             <max_speed>20</max_speed>
-            <max_steer>1.5</max_steer>
-            <max_steering_angle>9.0</max_steering_angle>
+            <max_steer>1.57</max_steer>
+            <max_steering_angle>15.0</max_steering_angle>
             <!-- PID tuning -->
             <left_steering_pid_gain>200 0 1</left_steering_pid_gain>

File: description/common.xacro (robot description, xacro)
@@ -1,5 +1,6 @@
 <?xml version="1.0"?>
 <robot xmlns:xacro="http://www.ros.org/wiki/xacro" >
-    <!-- This file contains the inertial macros used across the URDF files -->
+    <!-- This file contains the macros used across the URDF files -->
+    <!-- Inertial Macros -->
     <!-- Inertial Sphere Macros -->
     <xacro:macro name="inertial_sphere" params="mass radius *origin">
@@ -32,4 +33,28 @@
         </inertial>
     </xacro:macro>
-    <!-- Add more here -->
+    <!-- Material Macros -->
+    <material name="white">
+        <color rgba="1 1 1 1" />
+    </material>
+    <material name="orange">
+        <color rgba="1 0.3 0.1 1"/>
+    </material>
+    <material name="blue">
+        <color rgba="0.2 0.2 1 1"/>
+    </material>
+    <material name="black">
+        <color rgba="0 0 0 1"/>
+    </material>
+    <material name="red">
+        <color rgba="1 0 0 1"/>
+    </material>
+    <material name="grey">
+        <color rgba="0.631 0.631 0.631 1"/>
+    </material>
+    <material name="purple">
+        <color rgba="0.78 0.153 0.71 1"/>
+    </material>
+    <material name="green">
+        <color rgba="0.149 0.612 0.082 1"/>
+    </material>
 </robot>

File: description/depth_camera.xacro (robot description, xacro)
@@ -1,5 +1,5 @@
 <?xml version="1.0"?>
 <robot xmlns:xacro="http://www.ros.org/wiki/xacro" >
-    <!-- Deepth Camera -->
+    <!-- Depth Camera -->
     <joint name="camera_joint" type="fixed">
         <parent link="chassis"/>
@@ -15,5 +15,5 @@
         </visual>
     </link>
-    <!-- Deepth camera optical link -->
+    <!-- Depth camera optical link -->
     <joint name="camera_optical_joint" type="fixed">
         <parent link="camera_link"/>
@@ -22,5 +22,5 @@
     </joint>
     <link name="camera_link_optical"></link>
-    <!-- Deepth Camera Gazebo Sensor Plugin -->
+    <!-- Depth Camera Gazebo Sensor Plugin -->
     <gazebo reference="camera_link">
         <material>Gazebo/Purple</material>

File: description/diff_bot.urdf.xacro (robot description, xacro)
@@ -3,6 +3,5 @@
     <!-- Main URDF file for Differential Drive Robot -->
     <!-- Include general xacro files -->
-    <xacro:include filename="inertials.xacro"/>
-    <xacro:include filename="materials.xacro"/>
+    <xacro:include filename="common.xacro"/>
     <!-- Include sensors -->
     <xacro:include filename="lidar.xacro"/>

File: description/four_wheel.urdf.xacro (robot description, xacro)
@@ -3,6 +3,5 @@
     <!-- Main URDF file for Differential Drive Robot -->
     <!-- Include general xacro files -->
-    <xacro:include filename="inertials.xacro"/>
-    <xacro:include filename="materials.xacro"/>
+    <xacro:include filename="common.xacro"/>
     <!-- Include sensors -->
     <xacro:include filename="lidar.xacro"/>

Commit message: Updated models

File: description/ackermann.urdf.xacro (robot description, xacro)
@@ -10,13 +10,13 @@
     <!-- <xacro:include filename="3dlidar.xacro"/> -->
     <!-- Robot Variables -->
-    <xacro:property name="body_mass" value="20.0" />
+    <xacro:property name="chassis_mass" value="20.0" />
     <xacro:property name="wheel_mass" value="3.0" />
     <xacro:property name="steering_mass" value="0.01" />
-    <xacro:property name="body_length" value="0.35" />
-    <xacro:property name="body_width" value="0.3" />
-    <xacro:property name="body_heigth" value="0.08" />
+    <xacro:property name="chassis_length" value="0.35" />
+    <xacro:property name="chassis_width" value="0.3" />
+    <xacro:property name="chassis_heigth" value="0.08" />
     <xacro:property name="front_wheel_offset_x" value="0.15" />
     <xacro:property name="rear_wheel_offset_x" value="-0.15" />
-    <xacro:property name="wheel_offset_y" value="${body_width/2 + wheel_thickness/2}" />
+    <xacro:property name="wheel_offset_y" value="${chassis_width/2 + wheel_thickness/2}" />
     <xacro:property name="wheel_offset_z" value="0.0" />
     <xacro:property name="wheel_radius" value="0.05" />
@@ -39,17 +39,17 @@
     <link name="chassis">
         <visual>
-            <origin xyz="0 0 ${body_heigth/2}"/>
-            <geometry>
-                <box size="${body_length} ${body_width} ${body_heigth}"/>
+            <origin xyz="0 0 ${chassis_heigth/2}"/>
+            <geometry>
+                <box size="${chassis_length} ${chassis_width} ${chassis_heigth}"/>
             </geometry>
             <material name="purple"/>
         </visual>
         <collision>
-            <origin xyz="0 0 ${body_heigth/2}"/>
-            <geometry>
-                <box size="${body_length} ${body_width} ${body_heigth}"/>
-            </geometry>
-        </collision>
-        <xacro:inertial_box mass="${body_mass}" x="${body_length}" y="${body_width}" z="${body_heigth}">
+            <origin xyz="0 0 ${chassis_heigth/2}"/>
+            <geometry>
+                <box size="${chassis_length} ${chassis_width} ${chassis_heigth}"/>
+            </geometry>
+        </collision>
+        <xacro:inertial_box mass="${chassis_mass}" x="${chassis_length}" y="${chassis_width}" z="${chassis_heigth}">
             <origin xyz="0 0 0" rpy="0 0 0"/>
         </xacro:inertial_box>
@@ -61,5 +61,5 @@
         <origin xyz="${front_wheel_offset_x} ${wheel_offset_y} ${wheel_offset_z}" rpy="0 0 0" />
         <axis xyz="0 0 1" />
-        <limit upper="0.8" lower="-0.8" effort="-1.0" velocity="-1.0" />
+        <limit upper="0.6" lower="-0.6" effort="-1.0" velocity="-1.0" />
     </joint>
     <link name="front_left_steer">
@@ -80,5 +80,5 @@
         <origin xyz="${front_wheel_offset_x} ${-wheel_offset_y} ${wheel_offset_z}" rpy="0 0 0" />
         <axis xyz="0 0 1" />
-        <limit upper="0.8" lower="-0.8" effort="-1.0" velocity="-1.0" />
+        <limit upper="0.6" lower="-0.6" effort="-1.0" velocity="-1.0" />
     </joint>
     <link name="front_right_steer">
@@ -249,5 +249,5 @@
     <!-- Gazebo -->
     <gazebo reference="chassis">
-        <material>Gazebo/Blue</material>
+        <material>Gazebo/Purple</material>
     </gazebo>
     <gazebo reference="front_left_wheel">
@@ -269,5 +269,5 @@
     <gazebo>
         <plugin name='gazebo_ackermann_drive' filename='libgazebo_ros_ackermann_drive.so'>
-            <update_rate>100.0</update_rate>
+            <update_rate>60.0</update_rate>
             <!-- Wheels -->
             <front_left_joint>front_left_wheel_joint</front_left_joint>
